Commit message: add control plugin for the head. File .yaml added. Launch and urdf modified

File: src/exp_assignment2/urdf/robot.xacro (robot description, xacro)
@@ -241,3 +241,14 @@
 	    <child link="camera_link"/>
 	 </joint>
+<!-- Set trasmission for the head -->
+<transmission name="head_joint_trans">
+	<type>transmission_interface/SimpleTransmission</type>
+	<joint name="head_joint">
+		<hardwareInterface>hardware_interface/EffortJointInterface</hardwareInterface>
+	</joint>
+	<actuator name="motor1">
+		<hardwareInterface>hardware_interface/EffortJointInterface</hardwareInterface>
+		<mechanicalInterface>1</mechanicalInterface>
+	</actuator>
+</transmission>
 </robot>

Commit message: head motion fixed

File: src/exp_assignment2/urdf/robot.xacro (robot description, xacro)
@@ -240,5 +240,5 @@
 	    <parent link="head_link"/>
 	    <child link="camera_link"/>
-	 </joint>
+	</joint>
 <!-- Set trasmission for the head -->
 <transmission name="head_joint_trans">
